File: PXF_CAPE_PCB/PixHawk_Fire_v1.4.brd (EAGLE design)
At the start: 86.4 x 54.6 mm, 236 parts, among them J305 DF13-3P-1.25V, J306 DF13-4P-1.25V, J307 DF13-4P-1.25V, J308 DF13-4P-1.25V, J309 DF13-5P-1.25V, J310 DF13-4P-1.25V, J314 DF13-4P-1.25V, J701 JST-ZH-3, J801 DF13C-6P-1.25V, M3_MOUNT901 MOUNT-HOLE3.1MM, M3_MOUNT902 MOUNT-HOLE3.1MM, M3_MOUNT903 MOUNT-HOLE3.1MM, M3_MOUNT904 MOUNT-HOLE3.1MM, Q501 MMBT3906LT1SMD, U1 EEPROM-I2CSMD, U102 FM25V01, U2 EEPROM-I2CSMD, U201 TXS0108QFN20, U202 TXS0108QFN20, U301 MAX3051, U302 TXS0108QFN20, U303 PCA9306, U401 MS5611-01BA, U402 MS5611-01BA, U403 MPU-6000, U405 MPU-9250, U406 LSM9DS0LSM9DS0, U407 BMP280_PRELIM, U501 BQ24315, U502 MIC5332, U503 BQ24315, U601 TCA62724FMG, U602 LT3469, U603 LRTB GFTG-T7AW-1+V7A7-29+R5T9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, U701 TXS0108QFN20, U702 TXS0108QFN20, U703 74LVC2G240, U704 BBB_3X14_RA, U802 MIC5332, X801 4 pin head

Commit message: fixed missing ground on Serial 3 plug
Parts:
- removed U$10, U$13, U$14, U$15, U$5, U$6, U$7, U$8, U$9: CREATIVE_COMMONS, SparkFun:CREATIVE_COMMONS
Connections:
- net GND: now also U$3.6
Routing:
- net GND: track 410.1 -> 419.0 mm
Other:
- board text removed: "Direct cloning is NOT desired, but if you do.... please follow the spirit of OSHW, do not try and hide the fact that they are clones, do not expect that your cloned boards will interoperate with software designed for the original boards. for use in a flying vehicle, ensure that you have complied with any requirements found on Ardupilot.com in preparing the Certificate of Authenticity that will re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"
- board text removed: "Philip Rowse, 3D Robotics, Lorenz Meiers, and the PX4 team"
Changed lines of the file:
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@@
 <?xml version="1.0" encoding="utf-8"?>
 <!DOCTYPE eagle SYSTEM "eagle.dtd">
-<eagle version="6.5.0">
+<eagle version="6.6.0">
 <drawing>
 <settings>
@@
 <layer number="19" name="Unrouted" color="13" fill="1" visible="yes" active="yes"/>
 <layer number="20" name="Dimension" color="15" fill="1" visible="yes" active="yes"/>
-<layer number="21" name="tPlace" color="7" fill="1" visible="no" active="yes"/>
+<layer number="21" name="tPlace" color="7" fill="1" visible="yes" active="yes"/>
 <layer number="22" name="bPlace" color="7" fill="1" visible="no" active="yes"/>
 <layer number="23" name="tOrigins" color="15" fill="1" visible="yes" active="yes"/>
@@
 <wire x1="87.63" y1="8.636" x2="87.63" y2="8.128" width="0.15" layer="21"/>
 <wire x1="87.376" y1="8.382" x2="87.884" y2="8.382" width="0.15" layer="21"/>
-<text x="123.952" y="-80.01" size="1.778" layer="21">Philip Rowse, 3D Robotics, Lorenz Meiers, and the PX4 team</text>
-<text x="123.952" y="-71.374" size="1.778" layer="21">Philip Rowse, 3D Robotics, Lorenz Meiers, and the PX4 team</text>
-<text x="123.952" y="-62.738" size="1.778" layer="21">Philip Rowse, 3D Robotics, Lorenz Meiers, and the PX4 team</text>
-<text x="123.19" y="-54.356" size="1.778" layer="21">Philip Rowse, 3D Robotics, Lorenz Meiers, and the PX4 team</text>
-<text x="123.444" y="-45.974" size="1.778" layer="21">Philip Rowse, 3D Robotics, Lorenz Meiers, and the PX4 team</text>
-<text x="123.444" y="-36.83" size="1.778" layer="21">Philip Rowse, 3D Robotics, Lorenz Meiers, and the PX4 team</text>
-<text x="122.682" y="-28.448" size="1.778" layer="21">Philip Rowse, 3D Robotics, Lorenz Meiers, and the PX4 team</text>
-<text x="122.936" y="-20.066" size="1.778" layer="21">Philip Rowse, 3D Robotics, Lorenz Meiers, and the PX4 team</text>
-<text x="123.19" y="-11.176" size="1.778" layer="21">Philip Rowse, 3D Robotics, Lorenz Meiers, and the PX4 team</text>
-<text x="71.882" y="63.246" size="1.778" layer="21">Direct cloning is NOT desired, but if you do....
-please follow the spirit of OSHW, do not try and hide the fact that they are clones, do not expect that your cloned boards will interoperate with software designed for the original boards.
-for use in a flying vehicle, ensure that you have complied with any requirements found on Ardupilot.com in preparing the Certificate of Authenticity that will reside on the SHA chip on the board.
-if you make a clone or derivative of this board, you must release your exact schematics and PCB doccuments, and include these notices on every page.</text>
 </plain>
 <attributes>
@@
 <attribute name="BOM" value="EXCLUDE" x="123.952" y="33.528" size="1.778" layer="28" rot="MR180" display="off"/>
 </element>
-<element name="U$6" library="SparkFun" package="CREATIVE_COMMONS" value="CREATIVE_COMMONS" x="92.202" y="-10.922"/>
-<element name="U$5" library="SparkFun" package="CREATIVE_COMMONS" value="CREATIVE_COMMONS" x="92.202" y="-19.558"/>
-<element name="U$7" library="SparkFun" package="CREATIVE_COMMONS" value="CREATIVE_COMMONS" x="92.202" y="-28.194"/>
-<element name="U$8" library="SparkFun" package="CREATIVE_COMMONS" value="CREATIVE_COMMONS" x="92.202" y="-36.83"/>
-<element name="U$9" library="SparkFun" package="CREATIVE_COMMONS" value="CREATIVE_COMMONS" x="92.202" y="-45.466"/>
-<element name="U$10" library="SparkFun" package="CREATIVE_COMMONS" value="CREATIVE_COMMONS" x="92.202" y="-54.102"/>
-<element name="U$13" library="SparkFun" package="CREATIVE_COMMONS" value="CREATIVE_COMMONS" x="92.202" y="-62.738"/>
-<element name="U$14" library="SparkFun" package="CREATIVE_COMMONS" value="CREATIVE_COMMONS" x="92.202" y="-71.374"/>
-<element name="U$15" library="SparkFun" package="CREATIVE_COMMONS" value="CREATIVE_COMMONS" x="92.202" y="-80.01"/>
 <element name="C416" library="pixhawk2" package="0603-CAP" value="0u01" x="126.619" y="31.115" rot="MR180">
 <attribute name="PARTNO" value="06033C103JAT2A" x="126.619" y="30.861" size="1.778" layer="28" rot="MR180" display="off"/>
@@
 <wire x1="120.142" y1="22.479" x2="120.333" y2="22.479" width="0.15" layer="16"/>
 <wire x1="120.333" y1="22.479" x2="120.4364" y2="22.5824" width="0.15" layer="16"/>
+<contactref element="U$3" pad="6"/>
+<wire x1="81.7094" y1="22.973" x2="82.155" y2="22.973" width="0.254" layer="16"/>
+<wire x1="82.155" y1="22.973" x2="82.296" y2="23.114" width="0.4064" layer="16"/>
+<wire x1="82.296" y1="23.114" x2="82.3936" y2="23.114" width="0.4064" layer="16"/>
+<wire x1="82.3936" y1="23.114" x2="82.7214" y2="23.4418" width="0.4064" layer="16"/>
+<wire x1="108.635" y1="6.0215" x2="108.585" y2="6.0215" width="0.4064" layer="1"/>
+<wire x1="108.585" y1="6.0215" x2="108.585" y2="9.144" width="0.4064" layer="1"/>
+<wire x1="108.585" y1="9.144" x2="108.458" y2="9.144" width="0.4064" layer="1"/>
+<wire x1="108.458" y1="9.144" x2="107.95" y2="9.652" width="0.4064" layer="1"/>
+<wire x1="107.95" y1="9.652" x2="106.426" y2="9.652" width="0.4064" layer="1"/>
+<wire x1="106.426" y1="9.652" x2="106.172" y2="9.398" width="0.4064" layer="1"/>
+<wire x1="106.172" y1="9.398" x2="106.172" y2="8.128" width="0.4064" layer="1"/>
+<wire x1="106.0995" y1="8.636" x2="106.0995" y2="8.2005" width="0.4064" layer="1"/>
+<wire x1="106.0995" y1="8.2005" x2="106.172" y2="8.128" width="0.4064" layer="1"/>
 </signal>
 <signal name="BBB-VDD_3V3" class="1">
